File: Magnetic_field_profiler/Magnetic_field_profiler.kicad_sch (KiCad schematic)
At the start: 75 parts, among them J1 USB_B_Micro, J3 Conn_01x04_Socket, Q1 BSS123, SW1 SW_SPDT, U1 STM32F103C8Tx, U10 MLX90393, U11 MLX90393, U12 MLX90393, U13 TP6841S6, U3 DRV8825, U4 MLX90393, U5 MLX90393, U6 MLX90393, U7 MLX90393, U8 MLX90393, U9 MLX90393, Y1 Crystal_GND24

Commit message: PCB Updates and Second Motor Support
Parts:
- removed C17, C20, C21, C22, C23, C24, C25, C31, C32, C33, C34, C35, C36: 100n, Capacitor_SMD:C_0402_1005Metric, symbol Device:C
- removed U10, U11, U12, U4, U5, U6, U7, U8, U9: MLX90393, Package_DFN_QFN:QFN-16-1EP_3x3mm_P0.5mm_EP1.75x1.75mm_ThermalVias, symbol Mag_Profiler_ICs:MLX90393
- added J2: Conn_01x04_Socket, Connector_JST:JST_PH_S4B-PH-K_1x04_P2.00mm_Horizontal, symbol Connector:Conn_01x04_Socket
- added J4: Screw_Terminal_01x06, TerminalBlock:TerminalBlock_Xinya_XY308-2.54-6P_1x06_P2.54mm_Horizontal, symbol Connector:Screw_Terminal_01x06
- added R14: 1M, Resistor_SMD:R_0402_1005Metric, symbol Device:R
- added R15, R16, R17: 10k, Resistor_SMD:R_0402_1005Metric, symbol Device:R
- added R18: 50k, Resistor_SMD:R_0402_1005Metric, symbol Device:R
- added R19: 30k, Resistor_SMD:R_0402_1005Metric, symbol Device:R
- added R20, R21: 200m, Resistor_SMD:R_0402_1005Metric, symbol Device:R
- added U4: DRV8825, Package_SO:TSSOP-28-1EP_4.4x9.7mm_P0.65mm, symbol Mag_Profiler_ICs:DRV8825
- C14: value 100n -> 100u; footprint Capacitor_SMD:C_0402_1005Metric -> Capacitor_SMD:C_0805_2012Metric
- C16: value 100n -> 10n
Connections:
- net +12V: now also C12.1, C13.1, C14.1, C15.1, J4.4 (Pin_4), J4.5 (Pin_5), J4.6 (Pin_6), R14.1, U4.11 (VMB), U4.4 (VMA)
- net +3.3V: no longer C12.1, C13.1, C14.1, C15.1, C16.1
- net AVREF: now also R18.2, R19.1, U4.12 (AVREF), U4.13 (BVREF)
- net CP1: now also C16.1, U4.1 (CP1)
- net CP2: now also C16.2, U4.2 (CP2)
- net GND: now also J4.1 (Pin_1), J4.2 (Pin_2), J4.3 (Pin_3), R19.2, R20.2, R21.1, U4.14 (GND), U4.28 (GND), U4.29 (PPAD); no longer C15.2, C16.2
- net ISENA: now also R20.1, U4.6 (ISENA)
- net ISENB: now also R21.2, U4.9 (ISENB)
- net MTR_MODE0: now also U4.24 (MODE0)
- net MTR_MODE1: now also U4.25 (MODE1)
- net MTR_MODE2: now also U4.26 (MODE2)
- net MTR_NEN: now also U4.21 (nENABLE)
- net MTR_NRST: now also U4.16 (nRESET)
- net MTR_NSLEEP: now also R17.2, U4.17 (nSLEEP)
- net V3P3OUT: now also R17.1, R18.1; no longer R5.1, R6.1, U3.15 (V3P3OUT)
- net VCP: now also C15.2, R14.2, U4.3 (VCP)
- net MTR2_NFAULT: now reaches U1.13 (PA3)
- net MTR2_NFAULT: now also R15.2, U4.18 (nFAULT)
- net MTR2_NHOME: now reaches U1.14 (PA4)
- net MTR2_NHOME: now also R16.2, U4.27 (nHOME)
- net MTR2_DIR: now reaches U1.2 (PC13)
- net MTR2_DIR: now also U4.20 (DIR)
- net MTR2_STEP: now reaches U1.3 (PC14)
- net MTR2_STEP: now also U4.22 (STEP)
- net AOUT1 renamed M1_AOUT1
- net AOUT2 renamed M1_AOUT2
- net BOUT1 renamed M1_BOUT1
- net BOUT2 renamed M1_BOUT2
- net MTR_DIR renamed MTR1_DIR
- net MTR_NFAULT renamed MTR1_NFAULT
- net MTR_NHOME renamed MTR1_NHOME
- net MTR_STEP renamed MTR1_STEP
- new net M1_V3P3OUT: R5.1, R6.1, U3.15 (V3P3OUT)
- new net M2_AOUT1: J2.1 (Pin_1), U4.5 (AOUT1)
- new net M2_AOUT2: J2.2 (Pin_2), U4.7 (AOUT2)
- new net M2_BOUT1: J2.3 (Pin_3), U4.10 (BOUT1)
- new net M2_BOUT2: J2.4 (Pin_4), U4.8 (BOUT2)
- new net M2_V3P3OUT: R15.1, R16.1, U4.15 (V3P3OUT)
- no-connect marks 22 -> 10
Other:
- added sheet MAG1 (Magnetometer.kicad_sch)
- added sheet MAG2 (Magnetometer.kicad_sch)
- added sheet MAG3 (Magnetometer.kicad_sch)
- added sheet MAG4 (Magnetometer.kicad_sch)
- added sheet MAG5 (Magnetometer.kicad_sch)
- added sheet MAG6 (Magnetometer.kicad_sch)
- added sheet MAG7 (Magnetometer.kicad_sch)
- added sheet MAG8 (Magnetometer.kicad_sch)
- added sheet MAG9 (Magnetometer.kicad_sch)
- note added: "Power Input"
- note added: "Stepper Motor 1 Driver"
- note added: "Stepper Motor 2 Driver"
- note removed: "MAG (0,0)"
- note removed: "MAG (0,1)"
- note removed: "MAG (0,2)"
- note removed: "MAG (1,0)"
- note removed: "MAG (1,1)"
- note removed: "MAG (1,2)"
- note removed: "MAG (2,0)"
- note removed: "MAG (2,1)"
- note removed: "MAG (2,2)"
- note removed: "Stepper Motor Driver"
- moved on the sheet: Conn1, Q1, R1, R5, R6

Commit message: Symbol Properties Edits
Parts:
- removed J4: Screw_Terminal_01x06, TerminalBlock:TerminalBlock_Xinya_XY308-2.54-6P_1x06_P2.54mm_Horizontal, symbol Connector:Screw_Terminal_01x06
- added J4: Screw_Terminal_01x02, TerminalBlock_Phoenix:TerminalBlock_Phoenix_MKDS-1,5-2_1x02_P5.00mm_Horizontal, symbol Connector:Screw_Terminal_01x02
Connections:
- net +12V: now also J4.2 (Pin_2)
- net GND: now also J4.1 (Pin_1)

Commit message: MCU I2C configuration
Connections:
- net MAG_CS3: no longer U1.21 (PB10)
- net MAG_CS4: no longer U1.22 (PB11)
- new net I2C_SCL: U1.21 (PB10)
- new net I2C_SDA: U1.22 (PB11)
Changed lines of the file:
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@@
 	)
 	(bus_entry
-		(at 73.66 105.41)
-		(size -2.54 2.54)
-		(stroke
-			(width 0)
-			(type default)
-		)
-	)
-	(bus_entry
 		(at 226.06 72.39)
 		(size 2.54 2.54)
@@
 	)
 	(bus_entry
-		(at 73.66 102.87)
-		(size -2.54 2.54)
-		(stroke
-			(width 0)
-			(type default)
-		)
-	)
-	(bus_entry
 		(at 229.87 110.49)
 		(size 2.54 2.54)
@@
 		)
 	)
-	(bus
-		(pts
-			(xy 71.12 105.41) (xy 71.12 107.95)
-		)
-		(stroke
-			(width 0)
-			(type default)
-		)
-	)
 	(wire
 		(pts
@@
 	(bus
 		(pts
-			(xy 71.12 107.95) (xy 71.12 110.49)
+			(xy 71.12 85.09) (xy 71.12 110.49)
 		)
 		(stroke
@@
 		)
 	)
-	(bus
-		(pts
-			(xy 71.12 85.09) (xy 71.12 105.41)
-		)
-		(stroke
-			(width 0)
-			(type default)
-		)
-	)
 	(wire
 		(pts
@@
 		)
 	)
-	(label "MAG_CS3"
-		(at 73.66 102.87 0)
+	(label "MAG_CS9"
+		(at 59.69 118.11 0)
 		(fields_autoplaced yes)
 		(effects
@@
 		)
 	)
-	(label "MAG_CS9"
-		(at 59.69 118.11 0)
+	(label "I2C_SCL"
+		(at 73.66 102.87 0)
 		(fields_autoplaced yes)
 		(effects
@@
 		)
 	)
+	(label "I2C_SDA"
+		(at 73.66 105.41 0)
+		(fields_autoplaced yes)
+		(effects
+			(font
+				(size 1.27 1.27)
+			)
+			(justify left bottom)
+		)
+	)
 	(label "BVREF"
 		(at 180.34 187.96 0)
@@
 		)
 	)
-	(label "MAG_CS4"
-		(at 73.66 105.41 0)
-		(fields_autoplaced yes)
-		(effects
-			(font
-				(size 1.27 1.27)
-			)
-			(justify left bottom)
-		)
-	)

Commit message: IO expander wchematic and footprint updated. Adjusted the schematic representation of the magnetometer array.
Parts:
- added U?: MCP23S17, Package_SO:SSOP-28_5.3x10.2mm_P0.65mm, symbol Mag_Profiler_ICs:MCP23S17
Connections:
- net +3.3V: now also U?.9 (VDD)
- net GND: now also U?.10 (VSS)
- no-connect marks 10 -> 12
Other:
- added sheet MAG10 (Magnetometer.kicad_sch)
- added sheet MAG11 (Magnetometer.kicad_sch)
- added sheet MAG12 (Magnetometer.kicad_sch)
- added sheet MAG13 (Magnetometer.kicad_sch)
- added sheet MAG14 (Magnetometer.kicad_sch)
- added sheet MAG15 (Magnetometer.kicad_sch)
- added sheet MAG16 (Magnetometer.kicad_sch)
- moved on the sheet: C12, C13, C14, C15, C16, C26, C27, C28, C29, C30, C37, C38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

Commit message: IO expander connections complete and PCB layout restarted
Parts:
- added C58: 100n, Capacitor_SMD:C_0402_1005Metric, symbol Device:C
- gave numbers to parts that had none: 1
- renumbered C18 to C10, C19 to C11, C39 to C12, C37 to C13, C38 to C14, C40 to C15, C26 to C16, C27 to C17, C28 to C18, C12 to C19, C13 to C20, C14 to C21, C29 to C22, C15 to C23, C30 to C24, C16 to C25, C11 to C9, J4 to J2, J2 to J4, R2 to R1, R15 to R10, R16 to R11, R7 to R12, R17 to R13, R8 to R14, R18 to R15, R9 to R16, R19 to R17, R10 to R18, R20 to R19, R3 to R2, R11 to R20, R1 to R3, R12 to R4, R13 to R5, R4 to R6, R14 to R7, R5 to R8, R6 to R9, U13 to U2, U3 to U4, U4 to U5
Connections:
- net +3.3V: now also C58.1
- net GND: now also U3.15 (A0), U3.16 (A1), U3.17 (A2), C58.2
- net MAG_CS1: now also U3.21 (GPA0); no longer U1.19 (PB1)
- net MAG_CS10: now also U3.2 (GPB1)
- net MAG_CS11: now also U3.3 (GPB2)
- net MAG_CS12: now also U3.4 (GPB3)
- net MAG_CS13: now also U3.5 (GPB4)
- net MAG_CS14: now also U3.6 (GPB5)
- net MAG_CS15: now also U3.7 (GPB6)
- net MAG_CS16: now also U3.8 (GPB7)
- net MAG_CS2: now also U3.22 (GPA1); no longer U1.20 (PB2)
- net MAG_CS3: now also U3.23 (GPA2)
- net MAG_CS4: now also U3.24 (GPA3)
- net MAG_CS5: now also U3.25 (GPA4); no longer U1.25 (PB12)
- net MAG_CS6: now also U3.26 (GPA5); no longer U1.26 (PB13)
- net MAG_CS7: now also U3.27 (GPA6); no longer U1.29 (PA8)
- net MAG_CS8: now also U3.28 (GPA7); no longer U1.28 (PB15)
- net MAG_CS9: now also U3.1 (GPB0); no longer U1.27 (PB14)
- net SPI.SPI_CLK: now also U3.12 (SCK)
- net SPI.SPI_MISO: now also U3.14 (SO)
- net SPI.SPI_MOSI: now also U3.13 (SI)
- net IO_CS: now reaches U3.11 (CS)
- net IO_CS: now also U1.28 (PB15)
- net IO_RST: now reaches U3.18 (RESET)
- net IO_RST: now also U1.27 (PB14)
- net I2C_SCL: no longer names the net of U1.21 (PB10)
- net I2C_SDA: no longer names the net of U1.22 (PB11)
Other:
- moved on the sheet: U3
