File: Magnetic_field_profiler/Magnetic_field_profiler.kicad_sch (KiCad schematic)
At the start: 71 parts, among them J1 USB_B_Micro, J2 Screw_Terminal_01x02, J3 Conn_01x04_Socket, J4 Conn_01x04_Socket, Q1 BSS123, SW1 SW_SPDT, U1 STM32F103C8Tx, U2 AP63203WU, U3 MCP23S17, U4 DRV8825, U5 DRV8825, Y1 Crystal_GND24

Commit message: Initial PCB layout
Connections:
- net +5V: no longer names the net of J1.1 (VBUS)
- net IO_CS renamed IO1_CS
- net IO_RST renamed IO1_RST
- no-connect marks 18 -> 19
Changed lines of the file:
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@@
 	)
 	(no_connect
+		(at 149.86 69.85)
+	)
+	(no_connect
 		(at 118.11 74.93)
 	)
@@
 	(wire
 		(pts
-			(xy 148.59 62.23) (xy 148.59 69.85)
-		)
-		(stroke
-			(width 0)
-			(type default)
-		)
-	)
-	(wire
-		(pts
 			(xy 52.07 198.12) (xy 59.69 198.12)
 		)
@@
 		)
 	)
-	(wire
-		(pts
-			(xy 149.86 69.85) (xy 148.59 69.85)
-		)
-		(stroke
-			(width 0)
-			(type default)
-		)
-	)
 	(bus
 		(pts
@@
 		)
 	)
-	(label "IO_RST"
+	(label "IO1_RST"
 		(at 73.66 110.49 0)
 		(fields_autoplaced yes)
@@
 		)
 	)
-	(label "IO_CS"
+	(label "IO1_CS"
 		(at 311.15 165.1 0)
 		(fields_autoplaced yes)
@@
 		)
 	)
-	(label "IO_CS"
+	(label "IO1_CS"
 		(at 73.66 107.95 0)
 		(fields_autoplaced yes)
@@
 		)
 	)
-	(label "IO_RST"
+	(label "IO1_RST"
 		(at 311.15 160.02 0)
 		(fields_autoplaced yes)
@@
 					(unit 1)
 				)
-			)
-		)
-	)
-	(symbol
-		(lib_id "power:+5V")
-		(at 148.59 62.23 0)
-		(unit 1)
-		(exclude_from_sim no)
-		(in_bom yes)
-		(on_board yes)
-		(dnp no)
-		(fields_autoplaced yes)
-		(property "Reference" "#PWR011"
-			(at 148.59 66.04 0)
-			(effects
-				(font
-					(size 1.27 1.27)
-				)
-				(hide yes)
-			)
-		)
-		(property "Value" "+5V"
-			(at 148.59 57.15 0)
-			(effects
-				(font
-					(size 1.27 1.27)
-				)
-			)
-		)
-		(property "Footprint" ""
-			(at 148.59 62.23 0)
-			(effects
-				(font
-					(size 1.27 1.27)
-				)
-				(hide yes)
-			)
-		)
-		(property "Datasheet" ""
-			(at 148.59 62.23 0)
-			(effects
-				(font
-					(size 1.27 1.27)
-				)
-				(hide yes)
-			)
-		)
-		(property "Description" "Power symbol creates a global label with name \"+5V\""
-			(at 148.59 62.23 0)
-			(effects
-				(font
-					(size 1.27 1.27)
-				)
-				(hide yes)
-			)
-		)
-		(pin "1"
-		)
-		(instances
-			(project "Magnetic_field_profiler"
-				(path "/a3309886-ab27-4f3f-a056-7adffbf55c8a"
-					(reference "#PWR011")
-					(unit 1)
-				)
